Commit message: Aggiunto qualche task per l'action server e sistemate collisioni nella scena rviz

File: coppelia_moveit/config/ur5e_with_robotiq85.urdf.xacro (robot description, xacro)
@@ -8,5 +8,5 @@
     <xacro:ur5e_with_robotiq85_ros2_control name="FakeSystem" initial_positions_file="$(arg initial_positions_file)"/>
     <!-- Lab Table -->
-    <link name="lab_table">
+    <!-- <link name="lab_table">
         <visual>
             <origin xyz="0 0 0" rpy="0 0 0" />
@@ -31,4 +31,4 @@
         <child link="lab_table" />
         <origin xyz="0 0 0" rpy="0 0 0" />
-    </joint>
+    </joint> -->
 </robot>
